Commit message: add moveit config

File: phantomx_arm_description/urdf/pincher/pincher.urdf.xacro (robot description, xacro)
@@ -13,20 +13,29 @@
         <!-- Shoulder c-->
         <xacro:m_link name="${link_01_name}" o_rpy="0 0 ${M_PI_M}" o_xyz="0 0 0" geo_mesh="${geom_01_name}" mass="0.118" in_xyz="0.001031 -0.000032 -0.013806" ixx="0.030893" iyy="0.036432" izz="0.018984" ixy="0.000002" ixz="-0.000383" iyz="-0.000026" co_xyz="0 0 0" co_rpy="0 0 ${M_PI_M}" col_mesh="${colli_01_name}" />
-        <xacro:m_joint name="${joint_01_name}" type="revolute" origin_rpy="0 0 0" origin_xyz="0 0 0.137" parent="${link_00_name}" child="${link_01_name}" limit_e="1000.0" limit_l="-2.617993" limit_u="2.617993" limit_v="0.5" mimic="" mimic_joint=""/>
+        <xacro:m_joint name="${joint_01_name}" type="revolute" origin_rpy="0 0 0" origin_xyz="0 0 0.137" parent="${link_00_name}" child="${link_01_name}" limit_e="1000.0" limit_l="-2.617993" limit_u="2.617993" limit_v="1.5" mimic="" mimic_joint=""/>
         <!-- Lower arm -->
-        <xacro:m_link name="${link_02_name}" o_rpy="0 0 0" o_xyz="0 0 0" geo_mesh="${geom_02_name}" mass="0.162" in_xyz="0.080988 -0.000023 -0.000748" ixx="0.031204" iyy="0.124182" izz="0.111578" ixy="0.00002" ixz="0.001864" iyz="-0.000003" co_xyz="0 0 0" co_rpy="0 0 0" col_mesh="${colli_02_name}" />
-        <xacro:m_joint name="${joint_02_name}" type="revolute" origin_rpy="${M_PI_M} -${M_PI_M} 0" origin_xyz="0 0 0" parent="${link_01_name}" child="${link_02_name}" limit_e="1000.0" limit_l="-2.617993" limit_u="2.617993" limit_v="0.5" mimic="" mimic_joint=""/>
+        <xacro:m_link name="${link_02_name}" o_rpy="${M_PI} 0 0" o_xyz="0 0 0" geo_mesh="${geom_02_name}" mass="0.162" in_xyz="0.080988 -0.000023 -0.000748" ixx="0.031204" iyy="0.124182" izz="0.111578" ixy="0.00002" ixz="0.001864" iyz="-0.000003" co_xyz="0 0 0" co_rpy="${M_PI} 0 0" col_mesh="${colli_02_name}" />
+        <xacro:m_joint name="${joint_02_name}" type="revolute" origin_rpy="0 -${M_PI_M} -${M_PI_M}" origin_xyz="0 0 0" parent="${link_01_name}" child="${link_02_name}" limit_e="1000.0" limit_l="-2.617993" limit_u="2.617993" limit_v="1.5" mimic="" mimic_joint=""/>
         <!-- Upper arm -->
-        <xacro:m_link name="${link_03_name}" o_rpy="0 0 0" o_xyz="0 0 0" geo_mesh="${geom_03_name}" mass="0.162" in_xyz="0.080988 -0.000023 -0.000748" ixx="0.031204" iyy="0.124182" izz="0.111578" ixy="0.00002" ixz="0.001864" iyz="-0.000003" co_xyz="0 0 0" co_rpy="0 0 0" col_mesh="${colli_03_name}" />
-        <xacro:m_joint name="${joint_03_name}" type="revolute" origin_rpy="0 0 0" origin_xyz="0.105 0 0" parent="${link_02_name}" child="${link_03_name}" limit_e="1000.0" limit_l="-2.617993" limit_u="2.617993" limit_v="0.5" mimic="" mimic_joint=""/>
+        <xacro:m_link name="${link_03_name}" o_rpy="${M_PI} 0 0" o_xyz="0 0 0" geo_mesh="${geom_03_name}" mass="0.162" in_xyz="0.080988 -0.000023 -0.000748" ixx="0.031204" iyy="0.124182" izz="0.111578" ixy="0.00002" ixz="0.001864" iyz="-0.000003" co_xyz="0 0 0" co_rpy="${M_PI} 0 0" col_mesh="${colli_03_name}" />
+        <xacro:m_joint name="${joint_03_name}" type="revolute" origin_rpy="0 0 0" origin_xyz="0.105 0 0" parent="${link_02_name}" child="${link_03_name}" limit_e="1000.0" limit_l="-2.617993" limit_u="2.617993" limit_v="1.5" mimic="" mimic_joint=""/>
         <!-- wrist arm -->
-        <xacro:m_link name="${link_04_name}" o_rpy="0 0 0" o_xyz="0 0 0" geo_mesh="${geom_04_name}" mass="0.160" in_xyz="0.047054 0.009939 -0.000023" ixx="0.053897" iyy="0.057629" izz="0.068868" ixy="-0.002353" ixz="0.000011" iyz="0.000041" co_xyz="0 0 0" co_rpy="0 0 0" col_mesh="${colli_04_name}" />
-        <xacro:m_joint name="${joint_04_name}" type="revolute" origin_rpy="0 0 0" origin_xyz="0.105 0 0" parent="${link_03_name}" child="${link_04_name}" limit_e="1000.0" limit_l="-2.617993" limit_u="2.617993" limit_v="0.5" mimic="" mimic_joint=""/>
+        <xacro:m_link name="${link_04_name}" o_rpy="${M_PI} 0 0" o_xyz="0 0 0" geo_mesh="${geom_04_name}" mass="0.160" in_xyz="0.047054 0.009939 -0.000023" ixx="0.053897" iyy="0.057629" izz="0.068868" ixy="-0.002353" ixz="0.000011" iyz="0.000041" co_xyz="0 0 0" co_rpy="${M_PI} 0 0" col_mesh="${colli_04_name}" />
+        <xacro:m_joint name="${joint_04_name}" type="revolute" origin_rpy="0 0 0" origin_xyz="0.105 0 0" parent="${link_03_name}" child="${link_04_name}" limit_e="1000.0" limit_l="-2.617993" limit_u="2.617993" limit_v="1.5" mimic="" mimic_joint=""/>
+        <!-- gripper motor -->
+        <link name="gripper_revolute_link" />
+        <joint name="gripper_revolute_joint" type="revolute">
+            <parent link="${link_04_name}"/>
+            <child link="gripper_revolute_link"/>
+            <origin xyz="0.047 0 0" rpy="0 -${M_PI_M} 0"/>
+            <limit lower="-${M_PI}" upper="${M_PI}" effort="0" velocity="0"/>
+            <axis xyz="0 0 1"/>
+        </joint>
         <!-- Finger_1 -->
         <xacro:m_link name="${link_05_name}" o_rpy="0 0 0" o_xyz="0 0 0" geo_mesh="${geom_05_name}" mass="0.018" in_xyz="0.010769 0 -0.007406" ixx="0.002959" iyy="0.00287" izz="0.004524" ixy="0" ixz="-0.000707" iyz="0" co_xyz="0 0 0" co_rpy="0 0 0" col_mesh="${colli_05_name}" />
-        <xacro:m_joint name="${joint_05_name}" type="prismatic" origin_rpy="0 0 0" origin_xyz="0.071844 0 0" parent="${link_04_name}" child="${link_05_name}" limit_e="1000.0" limit_l="0" limit_u="0.015" limit_v="0.5" mimic="" mimic_joint=""/>
+        <xacro:m_joint name="${joint_05_name}" type="prismatic" origin_rpy="0 0 0" origin_xyz="0.071844 0 0" parent="${link_04_name}" child="${link_05_name}" limit_e="1000.0" limit_l="0" limit_u="0.015" limit_v="1.5" mimic="" mimic_joint=""/>
         <!-- Finger_2 -->
         <xacro:m_link name="${link_06_name}" o_rpy="0 0 0" o_xyz="0 0 0" geo_mesh="${geom_06_name}" mass="0.018" in_xyz="0.010769 0 -0.007406" ixx="0.002959" iyy="0.00287" izz="0.004524" ixy="0" ixz="-0.000707" iyz="0" co_xyz="0 0 0" co_rpy="0 0 0" col_mesh="${colli_06_name}" />
-        <xacro:m_joint name="${joint_06_name}" type="prismatic" origin_rpy="${M_PI} 0 0" origin_xyz="0.071844 0 0" parent="${link_04_name}" child="${link_06_name}" limit_e="1000.0" limit_l="0" limit_u="0.015" limit_v="0.5" mimic="1" mimic_joint="${joint_05_name}"/>
+        <xacro:m_joint name="${joint_06_name}" type="prismatic" origin_rpy="${M_PI} 0 0" origin_xyz="0.071844 0 0" parent="${link_04_name}" child="${link_06_name}" limit_e="1000.0" limit_l="0" limit_u="0.015" limit_v="1.5" mimic="1" mimic_joint="${joint_05_name}"/>
         <!-- Tool -->
         <link name="${link_07_name}">
